File: r6/src/_external_mic.kicad_sch (KiCad schematic)
At the start: 139 parts, among them Q12 BSS84PW, Q13 BSS84PW, Q14 NX3008NBKW, Q15 NX3008NBKW, Q16 NX3008NBKW, Q17 NX3008NBKW, Q18 NX3008NBKW, Q19 NX3008NBKW, Q20 BSS84PW, Q21 BSS84PW, Q22 NX3008NBKW, Q23 NX3008NBKW, Q24 NX3008NBKW, Q25 Si2323DS, Q29 Si2323DS, Q30 NX3008NBKW, T18 , T19 , T20 , T23 , T24 , T25 , T26 , T27 , T28 , T29 , T30 , T31 , T32 , T33 , T34 , T35 , T37 , T38 , T43 , T44 , T45 , T46 , T47 , T48 , T49 , T50 , T59 , U17 74HC20, U18 THAT5173, U19 74HC74, U20 74HC132, U21 74HC4520, U22 74HC132, U23 THAT1580, U24 74HC688, U25 LM4562, U26 74HC688, U27 AD4005, U36 APX809S-40SA

Commit message: r6: experimental revision of the r5 main board (unbuilt)
Filtered plug-in mic bias (R104 100R, Q25 supplied ahead of it),
4.7 nF ADC input filter, RV-3032 RTC on a new 3.3 V always-on rail,
Schmitt wake buffer, ADS1115 four-rail voltage monitoring, and a latched
modem SAFE_PWR_REMOVE/VGPIO shutdown confirmation (r5 erratum 5).

Outline, stack, all 37 fixed interfaces, USB and mic-input copper and
all r5 test points are unchanged. Designed and routed with AI coding
agents, reviewed by the author. No board has been built or measured.
Parts:
- C75, C76: value 180pF -> 4.7nF; MPN (none) -> GRM1555C1H472JE01D
Connections:
- net +3.3VA: no longer Q25.3 (D)
- new net R6_3V3_RAW: Q25.3 (D)
Other:
- note added: "R6: PIP supply RC filter R104/C83; Q25 bypasses R104 for P3V3 mode. C75/C76 = 4.7 nF C0G: 48 kHz population; validate SAR settling before release."
