File: r6/src/_modem.kicad_sch (KiCad schematic)
At the start: 59 parts, among them J1 , J12 U_FL-R-SMT-1_10_, J13 JAE_SIM_Card_SF72S006, J17 DNP, J2 , J3 , J4 , J5 , J6 , J7 , J8 , J9 , Q11 NX3008NBKW, Q5 NX3008NBKW, Q6 NX3008NBKW, Q7 NX3008NBKW, Q8 NX3008NBKW, Q9 NX3008NBKW, T10 , T11 , T4 , T55 , T56 , T57 , T58 , T8 , T9 , U7 Sierra_Wireless_RC7620, U8 ESD7004

Commit message: r6: experimental revision of the r5 main board (unbuilt)
Filtered plug-in mic bias (R104 100R, Q25 supplied ahead of it),
4.7 nF ADC input filter, RV-3032 RTC on a new 3.3 V always-on rail,
Schmitt wake buffer, ADS1115 four-rail voltage monitoring, and a latched
modem SAFE_PWR_REMOVE/VGPIO shutdown confirmation (r5 erratum 5).

Outline, stack, all 37 fixed interfaces, USB and mic-input copper and
all r5 test points are unchanged. Designed and routed with AI coding
agents, reviewed by the author. No board has been built or measured.
Connections:
- net R6_SAFE_RAW: now reaches U7.152 (SAFE_PWR_REMOVE)
- net R6_VGPIO_RAW: now reaches U7.45 (VGPIO)
- net J4: no longer names the net of J4.1, U7.239 (J4)
- no-connect marks 48 -> 46
