File: r6/src/_power.kicad_sch (KiCad schematic)
At the start: 176 parts, among them J10 502443-0860, Q1 Si7113ADN, Q10 Si2323DS, Q2 Si7113ADN, Q26 2SD1782KT146R, Q3 Si7113ADN, T1 , T12 , T13 , T17 , T2 , T21 , T22 , T36 , T41 , T42 , T5 , T51 , T52 , T6 , T7 , U2 ESD7004, U28 TPS65130RGE, U29 NCP163ASN330T1G, U3 DZDH0401DW, U30 NCP163ASN180T1G, U31 MAX6105, U32 LT8362xDD, U33 LM7121IM, U35 TPS22810DBV, U4 DZDH0401DW, U5 LM60440DRPK, U6 LM60440DRPK

Commit message: r6: experimental revision of the r5 main board (unbuilt)
Filtered plug-in mic bias (R104 100R, Q25 supplied ahead of it),
4.7 nF ADC input filter, RV-3032 RTC on a new 3.3 V always-on rail,
Schmitt wake buffer, ADS1115 four-rail voltage monitoring, and a latched
modem SAFE_PWR_REMOVE/VGPIO shutdown confirmation (r5 erratum 5).

Outline, stack, all 37 fixed interfaces, USB and mic-input copper and
all r5 test points are unchanged. Designed and routed with AI coding
agents, reviewed by the author. No board has been built or measured.
Parts:
- R104: value 0R -> 100R; MPN (none) -> RC0603FR-07100RL
Connections:
- net 3.3VA_O renamed R6_3V3_RAW
