File: r6/src/_sdcard.kicad_sch (KiCad schematic)
At the start: 6 parts, among them J14 Micro_SD_Card_Det_JAE_ST11, U10 ESD7004, U11 ESD7004

Commit message: r6: experimental revision of the r5 main board (unbuilt)
Filtered plug-in mic bias (R104 100R, Q25 supplied ahead of it),
4.7 nF ADC input filter, RV-3032 RTC on a new 3.3 V always-on rail,
Schmitt wake buffer, ADS1115 four-rail voltage monitoring, and a latched
modem SAFE_PWR_REMOVE/VGPIO shutdown confirmation (r5 erratum 5).

Outline, stack, all 37 fixed interfaces, USB and mic-input copper and
all r5 test points are unchanged. Designed and routed with AI coding
agents, reviewed by the author. No board has been built or measured.
Connections:
- no-connect marks 1 -> 0
Changed lines of the file:
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@@
 		(color 0 0 0 0)
-	)
-	(no_connect
-		(at 140.97 115.57)
 	)
 	(wire
@@
 		)
 		(instances
-			(project "bugg-main-r5"
+			(project "bugg-main-r6"
 				(path "/e3eb514f-6ce4-4abe-ba20-f82f0015628f/498d2354-7ecc-4881-a4b8-afc4730b4589"
 					(reference "J14")
@@
 		)
 		(instances
-			(project "bugg-main-r5"
+			(project "bugg-main-r6"
 				(path "/e3eb514f-6ce4-4abe-ba20-f82f0015628f/498d2354-7ecc-4881-a4b8-afc4730b4589"
 					(reference "#PWR0160")
@@
 		)
 		(instances
-			(project "bugg-main-r5"
+			(project "bugg-main-r6"
 				(path "/e3eb514f-6ce4-4abe-ba20-f82f0015628f/498d2354-7ecc-4881-a4b8-afc4730b4589"
 					(reference "R24")
@@
 		)
 		(instances
-			(project "bugg-main-r5"
+			(project "bugg-main-r6"
 				(path "/e3eb514f-6ce4-4abe-ba20-f82f0015628f/498d2354-7ecc-4881-a4b8-afc4730b4589"
 					(reference "C30")
@@
 		)
 		(instances
-			(project "bugg-main-r5"
+			(project "bugg-main-r6"
 				(path "/e3eb514f-6ce4-4abe-ba20-f82f0015628f/498d2354-7ecc-4881-a4b8-afc4730b4589"
 					(reference "#PWR0162")
@@
 		)
 		(instances
-			(project "bugg-main-r5"
+			(project "bugg-main-r6"
 				(path "/e3eb514f-6ce4-4abe-ba20-f82f0015628f/498d2354-7ecc-4881-a4b8-afc4730b4589"
 					(reference "C29")
@@
 		)
 		(instances
-			(project "bugg-main-r5"
+			(project "bugg-main-r6"
 				(path "/e3eb514f-6ce4-4abe-ba20-f82f0015628f/498d2354-7ecc-4881-a4b8-afc4730b4589"
 					(reference "#PWR0157")
@@
 		)
 		(instances
-			(project "bugg-main-r5"
+			(project "bugg-main-r6"
 				(path "/e3eb514f-6ce4-4abe-ba20-f82f0015628f/498d2354-7ecc-4881-a4b8-afc4730b4589"
 					(reference "#PWR0161")
@@
 		)
 		(instances
-			(project "bugg-main-r5"
+			(project "bugg-main-r6"
 				(path "/e3eb514f-6ce4-4abe-ba20-f82f0015628f/498d2354-7ecc-4881-a4b8-afc4730b4589"
 					(reference "U10")
@@
 		)
 		(instances
-			(project "bugg-main-r5"
+			(project "bugg-main-r6"
 				(path "/e3eb514f-6ce4-4abe-ba20-f82f0015628f/498d2354-7ecc-4881-a4b8-afc4730b4589"
 					(reference "#PWR0159")
@@
 		)
 		(instances
-			(project "bugg-main-r5"
+			(project "bugg-main-r6"
 				(path "/e3eb514f-6ce4-4abe-ba20-f82f0015628f/498d2354-7ecc-4881-a4b8-afc4730b4589"
 					(reference "U11")
@@
 		)
 		(instances
-			(project "bugg-main-r5"
+			(project "bugg-main-r6"
 				(path "/e3eb514f-6ce4-4abe-ba20-f82f0015628f/498d2354-7ecc-4881-a4b8-afc4730b4589"
 					(reference "#PWR0158")
