File: r6/src/bugg-main-r6.kicad_pcb (KiCad board)
At the start: 6 copper layers, 57.3 x 109 mm, 460 parts, among them J1 , J10 502443-0860, J12 U_FL-R-SMT-1_10_, J13 JAE_SIM_Card_SF72S006, J14 Micro_SD_Card_Det_JAE_ST11, J15 10118194, J16 FH12A-20S-0.5SH, J17 DNP, J2 , J3 , J4 , J5 , J6 , J7 , J8 , J9 , Q1 Si7113ADN, Q10 Si2323DS, Q11 NX3008NBKW, Q12 BSS84PW, Q13 BSS84PW, Q14 NX3008NBKW, Q15 NX3008NBKW, Q16 NX3008NBKW, Q17 NX3008NBKW, Q18 NX3008NBKW, Q19 NX3008NBKW, Q2 Si7113ADN, Q20 BSS84PW, Q21 BSS84PW, Q22 NX3008NBKW, Q23 NX3008NBKW, Q24 NX3008NBKW, Q25 Si2323DS, Q26 2SD1782KT146R, Q27 NX3008NBKW, Q28 NX3008NBKW, Q29 Si2323DS, Q3 Si7113ADN, Q30 NX3008NBKW, Q4 NX3008NBKW, Q5 NX3008NBKW, Q6 NX3008NBKW, Q7 NX3008NBKW, Q8 NX3008NBKW, Q9 NX3008NBKW, T1 , T10 , T11 , T12 , T13 , T14 , T15 , T16 , T17 , T18 , T19 , T2 , T20 , T21 , T22 , T23 , T24 , T25 , T26 , T27 , T28 , T29 , T3 , T30 , T31 , T32 , T33 , T34 , T35 , T36 , T37 , T38 , T39 , T4 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

Commit message: r6: experimental revision of the r5 main board (unbuilt)
Filtered plug-in mic bias (R104 100R, Q25 supplied ahead of it),
4.7 nF ADC input filter, RV-3032 RTC on a new 3.3 V always-on rail,
Schmitt wake buffer, ADS1115 four-rail voltage monitoring, and a latched
modem SAFE_PWR_REMOVE/VGPIO shutdown confirmation (r5 erratum 5).

Outline, stack, all 37 fixed interfaces, USB and mic-input copper and
all r5 test points are unchanged. Designed and routed with AI coding
agents, reviewed by the author. No board has been built or measured.
Parts:
- added C142: 1uF, Capacitor_SMD:C_0603_1608Metric, F.Cu at (-25.0, -14.8)
- added C143: 2.2uF, Capacitor_SMD:C_0603_1608Metric, F.Cu at (-25.5, -17.8)
- added C144: 100nF, Capacitor_SMD:C_0402_1005Metric, B.Cu at (-10.0, -29.6)
- added C145: 10nF, Capacitor_SMD:C_0402_1005Metric, F.Cu at (-4.50, -29.0)
- added C146: 10nF, Capacitor_SMD:C_0402_1005Metric, F.Cu at (-3.00, -29.0)
- added C147: 10nF, Capacitor_SMD:C_0402_1005Metric, F.Cu at (-1.50, -29.0)
- added C148: 10nF, Capacitor_SMD:C_0402_1005Metric, F.Cu at (0.00, -29.0)
- added C149: 100nF, Capacitor_SMD:C_0402_1005Metric, F.Cu at (9.50, -28.8)
- added C150: 100nF, Capacitor_SMD:C_0402_1005Metric, F.Cu at (26.8, -18.5)
- added C151: 100nF, Capacitor_SMD:C_0402_1005Metric, F.Cu at (26.5, -13.5)
- added Q31: BC847B,215, Package_TO_SOT_SMD:SOT-23, F.Cu at (15.5, -21.0)
- added Q32: BC847B,215, Package_TO_SOT_SMD:SOT-23, F.Cu at (17.0, -15.5)
- added R213: 150k, Resistor_SMD:R_0402_1005Metric, F.Cu at (-7.50, -28.0)
- added R214: 10k, Resistor_SMD:R_0402_1005Metric, F.Cu at (-5.90, -28.0)
- added R215: 20k, Resistor_SMD:R_0402_1005Metric, F.Cu at (-10.0, -31.5)
- added R216: 10k, Resistor_SMD:R_0402_1005Metric, F.Cu at (-8.90, -33.5)
- added R217: 10k, Resistor_SMD:R_0402_1005Metric, F.Cu at (-12.0, -32.0)
- added R218: 10k, Resistor_SMD:R_0402_1005Metric, F.Cu at (-8.90, -36.0)
- added R219: 20k, Resistor_SMD:R_0402_1005Metric, F.Cu at (-13.5, -32.0)
- added R220: 10k, Resistor_SMD:R_0402_1005Metric, F.Cu at (-8.90, -42.5)
- added R221: 47k, Resistor_SMD:R_0402_1005Metric, F.Cu at (10.0, -18.0)
- added R222: 470k, Resistor_SMD:R_0402_1005Metric, F.Cu at (14.0, -17.5)
- added R223: 10k, Resistor_SMD:R_0402_1005Metric, F.Cu at (16.0, -18.0)
- added R224: 47k, Resistor_SMD:R_0402_1005Metric, F.Cu at (12.0, -16.0)
- added R225: 470k, Resistor_SMD:R_0402_1005Metric, F.Cu at (14.0, -15.0)
- added R226: 10k, Resistor_SMD:R_0402_1005Metric, F.Cu at (16.0, -13.0)
- added R227: 10k, Resistor_SMD:R_0402_1005Metric, F.Cu at (12.0, -14.0)
- added R228: 100k, Resistor_SMD:R_0402_1005Metric, F.Cu at (14.0, -12.5)
- added U37: TPS7A0233PDBVR, Package_TO_SOT_SMD:SOT-23-5, F.Cu at (-22.0, -15.0)
- added U38: ADS1115IDGSR, Package_SO:MSOP-10_3x3mm_P0.5mm, F.Cu at (-11.5, -29.0)
- added U39: TCA9536DGKR, Package_SO:VSSOP-8_3x3mm_P0.65mm, F.Cu at (12.0, -27.0)
- added U40: SN74LVC1G74DCUR, Package_SO:VSSOP-8_2.3x2mm_P0.5mm, F.Cu at (24.0, -17.0)
- added U41: SN74LVC2G17DCKR, Package_TO_SOT_SMD:SOT-363_SC-70-6, F.Cu at (24.0, -12.5)
- C36: value 100nF -> 1uF
- C75, C76: value 180pF -> 4.7nF
- GC1, GC2, GC3, GC4: value TestPoint_Probe -> DNP
- J1, J2, J3, J4, J5, J6, J7, J8, J9, T1, T10, T11, T12, T13, T14, T15, T16, T17, T18, T19, T2, T20, T21, T22, T23, T24, T25, T26, T27, T28, T29, T3, T30, T31, T32, T33, T34, T35, T36, T37, T38, T39, T4, T40, T41, T42, T43, T44, T45, T46, T47, T48, T49, T5, T50, T51, T52, T53, T54, T55, T56, T57, T58, T59, T6, T7, T8, T9: value (none) -> ~
- R104: value 0R -> 100R
- R29: value 510k -> 100k
- R30: value 510k -> 47k
- U13: value DS3231MZ -> RV-3032-C7; footprint Package_SO:SOIC-8_3.9x4.9mm_P1.27mm -> Package_SON:MicroCrystal_C7_SON-8_1.5x3.2mm_P0.9mm
- U14: value 74LVC1G07DCK -> SN74LVC1G37DCKR
- turned U13 to 0 degrees
Connections:
- net /GLOBAL_EN_o renamed R6_GLOBAL_EN
- net /Modem/J4 renamed Net-(U7-J4)
- net /RTC/n_RTC_INT renamed R6_RTC_INT
- net /SCL renamed R6_SCL
- net Net-(C36-Pad1) renamed R6_WAKE_PULSE
- BT1 pad 1: /RTC/VBAT -> R6_VBAT
- C34 pad 1: /RTC/VBAT -> R6_VBAT
- C35 pad 1: +5V -> R6_AON3V3
- C98 pad 1: /Power and input connector/3.3VA_O -> R6_3V3_RAW
- D20 pad 2: /RTC/VBAT -> R6_VBAT
- J16 pad 17: /SDA -> R6_SDA
- Module1 pad 58: /SDA -> R6_SDA
- Q25 pad 3: +3.3VA -> R6_3V3_RAW
- Q28 pad 2: /SDA -> R6_SDA
- R104 pad 2: /Power and input connector/3.3VA_O -> R6_3V3_RAW
- R2 pad 1: /SDA -> R6_SDA
- R29 pad 1: +5V -> R6_AON3V3
- R30 pad 1: +5V -> R6_AON3V3
- T14 pad 1: /SDA -> R6_SDA
- T41 pad 1: /Power and input connector/3.3VA_O -> R6_3V3_RAW
- U11 pad 5: unconnected-(U11-IO4-Pad5) -> Net-(U11-IO4)
- U11 pad 6: unconnected-(U11-IO4-Pad5) -> Net-(U11-IO4)
- U13 pad 1: unconnected-(U13-32KHZ-Pad1) -> R6_VBAT
- U13 pad 2: +5V -> R6_SDA
- U13 pad 4: unconnected-(U13-~{RST}-Pad4) -> GND
- U13 pad 6: /RTC/VBAT -> R6_AON3V3
- U13 pad 7: /SDA -> unconnected-(U13-CLKOUT-Pad7)
- U14 pad 5: +5V -> R6_AON3V3
- U29 pad 5: /Power and input connector/3.3VA_O -> R6_3V3_RAW
- U7 pad 152: unconnected-(U7-SAFE_PWR_REMOVE-Pad152) -> R6_SAFE_RAW
- U7 pad 45: unconnected-(U7-VGPIO-Pad45) -> R6_VGPIO_RAW
Routing:
- net R6_SDA: track 0.00 -> 145.6 mm, vias 0 -> 11
- net +3V3: track 268.8 -> 371.5 mm, vias 13 -> 18
- net R6_SCL: track 76.2 -> 178.0 mm, vias 4 -> 9
- net GNDA: track 9.29 -> 105.9 mm
- net R6_VIN_SENSE: track 0.00 -> 88.9 mm, vias 0 -> 7
- net /SHDNZ: track 52.0 -> 139.3 mm, vias 2 -> 8
- net /SDA: track 83.7 -> 0.00 mm, vias 6 -> 0
- net R6_AON3V3: track 0.00 -> 70.7 mm, vias 0 -> 5
- net R6_LATCH_ARM: track 0.00 -> 67.8 mm, vias 0 -> 5
- net +3.3VADC: track 79.0 -> 146.7 mm, vias 21 -> 20
- net R6_SAFE_RAW: track 0.00 -> 62.1 mm, vias 0 -> 6
- net +5V: track 70.8 -> 130.5 mm, vias 35 -> 37
- net R6_3V7_SENSE: track 0.00 -> 59.0 mm, vias 0 -> 7
- net R6_VGPIO_RAW: track 0.00 -> 56.6 mm, vias 0 -> 3
- net IN_VIN: track 6.78 -> 61.8 mm, vias 12 -> 18
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- added copper zone on F.Cu, net R6_3V3_RAW
- removed copper zone on F.Cu, net /Power and input connector/3.3VA_O
Other:
- board text added: "bugg-main-r6-proto Monad 2023"
- board text removed: "bugg-main-r5 Monad 2023"
